File: kicad/greenhouse-control-unit/_autosave-greenhouse-control-unit.kicad_sch (KiCad schematic)
At the start: 39 parts, among them J1 Screw_Terminal_01x02, J10_Buck2 Conn_01x01_Female, J11_Buck2 Conn_01x01_Female, J12_Buck1 Conn_01x01_Female, J13_Buck1 Conn_01x01_Female, J14_Buck2 Conn_01x01_Female, J15_Buck2 Conn_01x01_Female, J16 Screw_Terminal_01x16, J2 Screw_Terminal_01x02, J3 Screw_Terminal_01x02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

Commit message: Add SR TTL, FET labels, tie PSU+12V to +12V
Parts:
- gave numbers to parts that had none: 1
Changed lines of the file:
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@@
   (symbol (lib_id "power:+5V") (at 271.78 160.02 0) (unit 1)
     (in_bom yes) (on_board yes) (fields_autoplaced)
-    (property "Reference" "#PWR?" (id 0) (at 271.78 163.83 0)
+    (property "Reference" "#PWR03" (id 0) (at 271.78 163.83 0)
       (effects (font (size 1.27 1.27)) hide)
     )
@@
   (symbol (lib_id "Nick:2N2222A") (at 269.24 165.1 0) (unit 1)
     (in_bom yes) (on_board yes) (fields_autoplaced)
-    (property "Reference" "Q?" (id 0) (at 274.32 163.8299 0)
+    (property "Reference" "Q8" (id 0) (at 274.32 163.8299 0)
       (effects (font (size 1.27 1.27)) (justify left))
     )
@@
       (reference "#PWR02") (unit 1) (value "GND") (footprint "")
     )
+    (path "/db6607a5-d24c-4fdf-98bd-7c48dca4f9ad"
+      (reference "#PWR03") (unit 1) (value "+5V") (footprint "")
+    )
     (path "/89f6aa24-278b-41b4-bb3b-e1e585067bd1"
       (reference "#PWR0101") (unit 1) (value "GND") (footprint "")
@@
       (reference "#PWR0125") (unit 1) (value "GND") (footprint "")
     )
-    (path "/db6607a5-d24c-4fdf-98bd-7c48dca4f9ad"
-      (reference "#PWR?") (unit 1) (value "+5V") (footprint "")
-    )
     (path "/e9cc145f-bccc-4781-862a-a53065926266"
       (reference "BZ1") (unit 1) (value "Buzzer") (footprint "Buzzer_Beeper:Buzzer_12x9.5RM7.6")
@@
     )
     (path "/ea36a4ae-b6e4-4966-a53d-e362137e93ee"
-      (reference "Q?") (unit 1) (value "2N2222A") (footprint "Package_TO_SOT_THT:TO-92_Inline")
+      (reference "Q8") (unit 1) (value "2N2222A") (footprint "Package_TO_SOT_THT:TO-92_Inline")
     )
     (path "/ded41c74-3323-47f8-b02d-55f1d484132e"
