File: kicad/greenhouse-control-unit/greenhouse-control-unit.kicad_sch (KiCad schematic)
At the start: 44 parts, among them J1 Screw_Terminal_01x02, J10 Conn_01x15_Female, J10_LittleBuck1 Conn_01x01_Female, J11 Conn_01x02_Male, J11_LittleBuck1 Conn_01x01_Female, J12 Screw_Terminal_01x16, J12_BigBuck1 Conn_01x01_Female, J13_BigBuck1 Conn_01x01_Female, J14_LittleBuck1 Conn_01x01_Female, J15_LittleBuck1 Conn_01x01_Female, J2 Screw_Terminal_01x02, J3 Screw_Terminal_01x02, J4 Screw_Terminal_01x02, J5 Screw_Terminal_01x02, J6 Screw_Terminal_01x02, J6_BigBuck1 Conn_01x01_Female, J7 Screw_Terminal_01x02, J7_BigBuck1 Conn_01x01_Female, J8 Conn_01x03_Male, J9 Conn_01x15_Female, Q1 IRLB8721PBF, Q2 2N2222A, Q3 2N2222A, Q4 2N2222A, Q5 IRLB8721PBF, Q6 IRLB8721PBF, Q7 IRLB8721PBF, Q8 IRLB8721PBF, U1 74HC595, U2 74HC595

Commit message: Add PSU diode, reorganize PCB layout
Parts:
- removed J6, J7: Screw_Terminal_01x02, TerminalBlock_Phoenix:TerminalBlock_Phoenix_MKDS-1,5-2-5.08_1x02_P5.08mm_Horizontal, symbol Connector:Screw_Terminal_01x02
- added D1: D_Schottky, Package_TO_SOT_THT:TO-126-2_Vertical, symbol Device:D_Schottky
- added D2, D4: LED, LED_THT:LED_D5.0mm, symbol Device:LED
- added J13: Conn_01x10_Female, Connector_Molex:Molex_KK-254_AE-6410-10A_1x10_P2.54mm_Vertical, symbol Connector:Conn_01x10_Female
- added J7, J8: Conn_01x10_Female, Connector_PinSocket_2.54mm:PinSocket_1x10_P2.54mm_Vertical, symbol Connector:Conn_01x10_Female
- added R1, R3: 5k, Resistor_THT:R_Axial_DIN0207_L6.3mm_D2.5mm_P7.62mm_Horizontal, symbol Device:R
- added R2, R4, R5, R6: 10k, Resistor_THT:R_Axial_DIN0207_L6.3mm_D2.5mm_P7.62mm_Horizontal, symbol Device:R
- added R8: 2k, Resistor_THT:R_Axial_DIN0207_L6.3mm_D2.5mm_P7.62mm_Horizontal, symbol Device:R
- J10, J9: footprint Connector_PinHeader_2.54mm:PinHeader_1x15_P2.54mm_Vertical -> Connector_PinSocket_2.54mm:PinSocket_1x15_P2.54mm_Vertical
- J12_BigBuck1, J13_BigBuck1, J6_BigBuck1, J7_BigBuck1: footprint Connector_PinHeader_2.54mm:PinHeader_1x01_P2.54mm_Vertical -> Connector_PinSocket_2.54mm:PinSocket_1x01_P2.54mm_Vertical
- R10: renamed from R5; footprint Resistor_THT:R_Box_L13.0mm_W4.0mm_P9.00mm -> Resistor_THT:R_Axial_DIN0207_L6.3mm_D2.5mm_P7.62mm_Horizontal
- R11: renamed from R2; value 10k -> 2k; footprint Resistor_THT:R_Box_L8.4mm_W2.5mm_P5.08mm -> Resistor_THT:R_Axial_DIN0207_L6.3mm_D2.5mm_P7.62mm_Horizontal
- R12: renamed from R3; value 10k -> 2k; footprint Resistor_THT:R_Box_L8.4mm_W2.5mm_P5.08mm -> Resistor_THT:R_Axial_DIN0207_L6.3mm_D2.5mm_P7.62mm_Horizontal
- R13: renamed from R6; footprint Resistor_THT:R_Box_L8.4mm_W2.5mm_P5.08mm -> Resistor_THT:R_Axial_DIN0207_L6.3mm_D2.5mm_P7.62mm_Horizontal
- R14: renamed from R7; footprint Resistor_THT:R_Box_L8.4mm_W2.5mm_P5.08mm -> Resistor_THT:R_Axial_DIN0207_L6.3mm_D2.5mm_P7.62mm_Horizontal
- R15: renamed from R8; footprint Resistor_THT:R_Box_L8.4mm_W2.5mm_P5.08mm -> Resistor_THT:R_Axial_DIN0207_L6.3mm_D2.5mm_P7.62mm_Horizontal
- R16: renamed from R9; footprint Resistor_THT:R_Box_L8.4mm_W2.5mm_P5.08mm -> Resistor_THT:R_Axial_DIN0207_L6.3mm_D2.5mm_P7.62mm_Horizontal
- R7: renamed from R1; footprint Resistor_THT:R_Box_L13.0mm_W4.0mm_P9.00mm -> Resistor_THT:R_Axial_DIN0207_L6.3mm_D2.5mm_P7.62mm_Horizontal
- R9: renamed from R4; footprint Resistor_THT:R_Box_L8.4mm_W2.5mm_P5.08mm -> Resistor_THT:R_Axial_DIN0207_L6.3mm_D2.5mm_P7.62mm_Horizontal
- renumbered D1 to D3, D4 to D5, D2 to D6, D3 to D7, J8 to J6
Connections:
- net BattRelayNC_Boil is gone; now on net BattRelayNC_Coil: Q1.2 (D)
- net +12V: now also J3.1 (Pin_1), J5.1 (Pin_1), D1.1 (K), R3.1, R5.1
- net +5VA: now also J9.1 (Pin_1), J13.1 (Pin_1), J7.1 (Pin_1), J8.1 (Pin_1); no longer J9.15 (Pin_15)
- net Batt+12V: now also J2.1 (Pin_1), J3.2 (Pin_2); no longer J2.2 (Pin_2), J3.1 (Pin_1)
- net BattRelayNC_Coil: now also J4.1 (Pin_1); no longer J4.2 (Pin_2)
- net BattRelayNC_SR_Q0: now also R8.1
- net GND: now also J1.2 (Pin_2), J2.2 (Pin_2), J4.2 (Pin_2), J5.2 (Pin_2), J9.2 (Pin_2), D2.1 (K), D4.1 (K), J13.3 (Pin_3), J7.2 (Pin_2), J8.2 (Pin_2), R2.2, R4.2, R6.2; no longer J1.1 (Pin_1), J2.1 (Pin_1), J4.1 (Pin_1), J5.1 (Pin_1), J9.14 (Pin_14)
- net MC_A0: now also J9.15 (Pin_15); no longer J9.1 (Pin_1)
- net MC_D3: now also J13.6 (Pin_6)
- net MC_D0: now reaches J10.15 (Pin_15)
- net MC_D0: now also R7.2, U1.13 (~{OE}), U2.13 (~{OE})
- removed net BattRelayNC_B: J1.2 (Pin_2), J3.2 (Pin_2), J5.2 (Pin_2)
- net I2C_SCL renamed ADC1_SCL
- net ADC1_SCL: now also J13.4 (Pin_4), J7.3 (Pin_3), J8.3 (Pin_3)
- net I2C_SDA renamed ADC1_SCA
- net ADC1_SCA: now also J13.5 (Pin_5), J7.4 (Pin_4), J8.4 (Pin_4)
- removed net MC_D8: J10.1 (Pin_1), R7.2, U1.13 (~{OE}), U2.13 (~{OE})
- new net: D2.2 (A), R5.2
- new net: D4.2 (A), R8.2
- new net +3V3: J10.1 (Pin_1), J13.2 (Pin_2)
- new net ADC1_A0: J13.7 (Pin_7), J7.7 (Pin_7)
- new net ADC1_A1: J13.8 (Pin_8), J7.8 (Pin_8)
- new net ADC1_A2: J13.9 (Pin_9), J7.9 (Pin_9)
- new net ADC1_A3: J13.10 (Pin_10), J7.10 (Pin_10)
- new net ADC1_ADDR: J7.5 (Pin_5)
- new net ADC1_ALRT: J7.6 (Pin_6)
- new net ADC2_A0: J8.7 (Pin_7), R3.2, R4.1
- new net ADC2_A1: J8.8 (Pin_8), R1.2, R2.1
- new net ADC2_A2: J8.9 (Pin_9)
- new net ADC2_A3: J8.10 (Pin_10)
- new net ADC2_ADDR: J8.5 (Pin_5), R6.1
- new net ADC2_ALRT: J8.6 (Pin_6)
- new net PSU+12V: D1.2 (A), J1.1 (Pin_1), R1.1
Other:
- note added: "Prototype TODO: - Power both relays from combined 12V power - Reduce sensor pin headers to single block - Swap out DPST relay for SPST relay - Add easy-disconnect terminals (x6) - Try PSU relay without BJT - Investigate diode on batt relay FET source (why?) - Reverse MC direction (rotate 90deg) - Move motor control pins to SR (remove PCF expander) - Add extra ADC - Change COM LED resistor to 10k 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"
- note added: "Schematic TODO: None"
- note added: "Sets address"
- note removed: "Prototype TODO: - Power both relays from combined 12V power - Reduce sensor pin headers to single block - Swap out DPST relay for SPST relay - Add easy-disconnect terminals (x6) - Try PSU relay without BJT - Investigate diode on batt relay FET source (why?) - Reverse MC direction (rotate 90deg)"
- note removed: "Schematic TODO: - Diode/FET to block battery/PSU connection - Voltage sensor/divider behind PSU diode"
- moved on the sheet: BZ1, D5, D6, D7, J11, J6, Q1, Q2, Q3, Q4, R10, R11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

Commit message: Connect relay coil to VCC, fixed footprints
Parts:
- removed J5: Screw_Terminal_01x02, TerminalBlock_Phoenix:TerminalBlock_Phoenix_MKDS-1,5-2-5.08_1x02_P5.08mm_Horizontal, symbol Connector:Screw_Terminal_01x02
- added J5: Conn_01x02_Male, Connector_Molex:Molex_KK-254_AE-6410-02A_1x02_P2.54mm_Vertical, symbol Connector:Conn_01x02_Male
- D1: value D_Schottky -> DSB20I15PA Schottky
- J13: symbol Connector:Conn_01x10_Female -> Connector:Conn_01x10_Male
Connections:
- net +12V: now also J4.2 (Pin_2), J5.1 (Pin_1)
- net GND: now also J5.2 (Pin_2); no longer J4.2 (Pin_2)
Other:
- moved on the sheet: J4

Commit message: R values, rearrange SRs on PCB
Parts:
- added J14: Conn_01x03_Male, Connector_Molex:Molex_KK-254_AE-6410-03A_1x03_P2.54mm_Vertical, symbol Connector:Conn_01x03_Male
- added R17: 4k6, Resistor_THT:R_Axial_DIN0207_L6.3mm_D2.5mm_P7.62mm_Horizontal, symbol Device:R
- R1, R3: value 5k -> 4k6
- R10: value R4k6 -> 4k6
- R13, R14, R15, R16, R7, R9: value R10k -> 10k
- R2, R4: value 10k -> 1k
Connections:
- net +3V3: now also J13.1 (Pin_1), J14.1 (Pin_1), R17.1; no longer J13.2 (Pin_2)
- net +5VA: no longer J13.1 (Pin_1)
- net GND: now also J13.2 (Pin_2); no longer J13.3 (Pin_3)
- net MC_D3: now also R17.2
- net SR_Q6 renamed Motor_IN1
- net Motor_IN1: now also J14.2 (Pin_2)
- net SR_Q7 renamed Motor_IN2
- net Motor_IN2: now also J14.3 (Pin_3)
Other:
- note added: "Prototype TODO: - Reduce sensor pin headers to single block - Add easy-disconnect terminals (x6) - Try PSU relay without BJT - Reverse MC direction (rotate 90deg) - Move motor control pins to SR (remove PCF expander) - Add extra ADC - Change relay LED to 2k - Replace fan and relay FETs with N27000"
- note added: "Schematic TODO: Replace BJTs with 2N7000 MOSFETs Replace relay IRLB with 2N7000"
- note removed: "Prototype TODO: - Power both relays from combined 12V power - Reduce sensor pin headers to single block - Swap out DPST relay for SPST relay - Add easy-disconnect terminals (x6) - Try PSU relay without BJT - Investigate diode on batt relay FET source (why?) - Reverse MC direction (rotate 90deg) - Move motor control pins to SR (remove PCF expander) - Add extra ADC - Change COM LED resistor to 10k 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"
- note removed: "Schematic TODO: None"
- moved on the sheet: D3, R7, U1, U2
