File: kicad/greenhouse-control-unit/greenhouse-control-unit.kicad_sch (KiCad schematic)
At the start: 69 parts, among them J1 Pluggable_Terminal_01x02, J10 Molex_KK-254_01x10, J10_LittleBuck1 Conn_01x01_Female, J11_LittleBuck1 Conn_01x01_Female, J12_BigBuck1 Conn_01x01_Female, J13_BigBuck1 Conn_01x01_Female, J14_LittleBuck1 Conn_01x01_Female, J15_LittleBuck1 Conn_01x01_Female, J2 Pluggable_Terminal_01x02, J3 Pluggable_Terminal_01x02, J4 Molex_KK-254_01x08, J5 Conn_01x10_Female, J6 Conn_01x10_Female, J6_BigBuck1 Conn_01x01_Female, J7 Conn_01x15_Female, J7_BigBuck1 Conn_01x01_Female, J8 Conn_01x15_Female, J9 Molex_KK-396_01x16, Q1 2N7000, Q10 IRLB8721PBF, Q11 IRLB8721PBF, Q2 2N7000, Q3 2N7000, Q4 IRLB8721PBF, Q5 IRLB8721PBF, Q6 IRLB8721PBF, Q7 IRLB8721PBF, Q8 IRLB8721PBF, Q9 IRLB8721PBF, U1 74HC595, U2 74HC595

Commit message: Updated TODOs
Other:
- note added: "Prototype TODO: - Consolidate several 2/3 headers into one - Change actuator controller header to 2 pin (split 1-2 to EN1-4) - Add LED to case fan FET - Check all R values - Test current on each SR out (max 20mA, limit 35mA) - Test current on SR VCC (max 70mA)"
- note added: "Schematic TODO: - Find less powerful 5V FET than IRLBx (but not 2N7000; max 3.5VGS) - Revert new FETs back to BJTs (which actually work fine)"
- note removed: "Prototype TODO: - Consolidate several 2/3 headers into one - Change actuator controller header to 4 pin (IN1-4, no EN) - Move relay LED to source - Add LED to case fan FET - Change relay LED to 2k - Check all R values - Test current on each SR out (max 20mA, limit 35mA) - Test current on SR VCC (max 70mA)"
- note removed: "Schematic TODO: - Find less powerful 5V FET than IRLBx (but not 2N7000; max 3.5VGS)"
Changed lines of the file:
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@@
     (effects (font (size 1.27 1.27)) (justify left bottom))
   )
-  (text "Schematic TODO:\n- Find less powerful 5V FET than IRLBx (but not 2N7000; max 3.5VGS)"
+  (text "Schematic TODO:\n- Find less powerful 5V FET than IRLBx (but not 2N7000; max 3.5VGS)\n- Revert new FETs back to BJTs (which actually work fine)"
     (at 107.95 24.13 0)
     (effects (font (size 1.27 1.27)) (justify left bottom))
   )
-  (text "Prototype TODO:\n- Consolidate several 2/3 headers into one\n- Change actuator controller header to 4 pin (IN1-4, no EN)\n- Move relay LED to source\n- Add LED to case fan FET\n- Change relay LED to 2k\n- Check all R values\n- Test current on each SR out (max 20mA, limit 35mA)\n- Test current on SR VCC (max 70mA)"
+  (text "Prototype TODO:\n- Consolidate several 2/3 headers into one\n- Change actuator controller header to 2 pin (split 1-2 to EN1-4)\n- Add LED to case fan FET\n- Check all R values\n- Test current on each SR out (max 20mA, limit 35mA)\n- Test current on SR VCC (max 70mA)"
     (at 26.67 36.83 0)
     (effects (font (size 1.27 1.27)) (justify left bottom))
