File: kicad/greenhouse-control-unit/greenhouse-control-unit.kicad_sch (KiCad schematic)
At the start: 69 parts, among them J1 Pluggable_Terminal_01x02, J10 Molex_KK-254_01x10, J10_LittleBuck1 Conn_01x01_Female, J11_LittleBuck1 Conn_01x01_Female, J12_BigBuck1 Conn_01x01_Female, J13_BigBuck1 Conn_01x01_Female, J14_LittleBuck1 Conn_01x01_Female, J15_LittleBuck1 Conn_01x01_Female, J2 Pluggable_Terminal_01x02, J3 Pluggable_Terminal_01x02, J4 Molex_KK-254_01x08, J5 Conn_01x10_Female, J6 Conn_01x10_Female, J6_BigBuck1 Conn_01x01_Female, J7 Conn_01x15_Female, J7_BigBuck1 Conn_01x01_Female, J8 Conn_01x15_Female, J9 Molex_KK-396_01x16, Q1 2N7000, Q10 IRLB8721PBF, Q11 IRLB8721PBF, Q2 2N7000, Q3 2N2222A, Q4 IRLB8721PBF, Q5 IRLB8721PBF, Q6 IRLB8721PBF, Q7 IRLB8721PBF, Q8 IRLB8721PBF, Q9 IRLB8721PBF, U1 74HC595, U2 74HC595

Commit message: Change cap for motor driver regulator
Also moved battery coil to PSU #236
Connections:
- net PSU+12V is gone; now on net BattRelayNC_Coil: D1.2 (A), J1.1 (Pin_1), R1.1
Other:
- note added: "Prototype TODO: - Swithc out L7805 for L7810 (motor driver supply FET driver) - Check all R values - Test current on each SR out (max 20mA, limit 35mA) - Test current on SR VCC (max 70mA)"
- note removed: "Prototype TODO: - Check all R values - Test current on each SR out (max 20mA, limit 35mA) - Test current on SR VCC (max 70mA) - Add EN transistor for SR - Add L298 to main board"
Changed lines of the file:
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@@
     (stroke (width 0) (type default) (color 0 0 0 0))
   )
-  (wire (pts (xy 91.44 148.59) (xy 109.22 148.59))
+  (wire (pts (xy 91.44 148.59) (xy 121.92 148.59))
     (stroke (width 0) (type default) (color 0 0 0 0))
   )
@@
     (stroke (width 0) (type default) (color 0 0 0 0))
   )
-  (wire (pts (xy 118.11 146.05) (xy 118.11 147.32))
-    (stroke (width 0) (type default) (color 0 0 0 0))
-  )
   (wire (pts (xy 157.48 134.62) (xy 170.18 134.62))
     (stroke (width 0) (type default) (color 0 0 0 0))
@@
     (stroke (width 0) (type default) (color 0 0 0 0))
   )
+  (wire (pts (xy 124.46 146.05) (xy 124.46 152.4))
+    (stroke (width 0) (type default) (color 0 0 0 0))
+  )
   (wire (pts (xy 332.74 151.13) (xy 342.9 151.13))
     (stroke (width 0) (type default) (color 0 0 0 0))
@@
     (stroke (width 0) (type default) (color 0 0 0 0))
   )
-  (wire (pts (xy 91.44 146.05) (xy 118.11 146.05))
+  (wire (pts (xy 91.44 146.05) (xy 124.46 146.05))
     (stroke (width 0) (type default) (color 0 0 0 0))
   )
@@
     (effects (font (size 1.27 1.27)) (justify left bottom))
   )
-  (text "Schematic TODO: \n- Disable SR when no input voltage (SR can draw power from inputs; i.e. MC)"
+  (text "Schematic TODO: \n- Disable SR when no input voltage (SR can draw power from inputs; i.e. MC)\n"
     (at 132.08 26.67 0)
     (effects (font (size 1.27 1.27)) (justify left bottom))
   )
-  (text "Prototype TODO:\n- Check all R values\n- Test current on each SR out (max 20mA, limit 35mA)\n- Test current on SR VCC (max 70mA)\n- Add EN transistor for SR\n- Add L298 to main board"
+  (text "Prototype TODO:\n- Swithc out L7805 for L7810 (motor driver supply FET driver)\n\n- Check all R values\n- Test current on each SR out (max 20mA, limit 35mA)\n- Test current on SR VCC (max 70mA)\n"
     (at 26.67 36.83 0)
     (effects (font (size 1.27 1.27)) (justify left bottom))
@@
     (effects (font (size 1.27 1.27)) (justify right bottom))
   )
+  (label "PSU+12V" (at 121.92 148.59 180)
+    (effects (font (size 1.27 1.27)) (justify right bottom))
+  )
   (label "SW_FET7" (at 368.3 113.03 0)
     (effects (font (size 1.27 1.27)) (justify left bottom))
@@
     (effects (font (size 1.27 1.27)) (justify right bottom))
   )
-  (symbol (lib_id "power:GND") (at 118.11 147.32 0) (unit 1)
-    (in_bom yes) (on_board yes)
-    (property "Reference" "#PWR06" (id 0) (at 118.11 153.67 0)
-      (effects (font (size 1.27 1.27)) hide)
-    )
-    (property "Value" "GND" (id 1) (at 118.11 152.4 0))
-    (property "Footprint" "" (id 2) (at 118.11 147.32 0)
-      (effects (font (size 1.27 1.27)) hide)
-    )
-    (property "Datasheet" "" (id 3) (at 118.11 147.32 0)
-      (effects (font (size 1.27 1.27)) hide)
-    )
-    (pin "1")
-  )
   (symbol (lib_id "Connector:Conn_01x01_Female") (at 107.95 114.3 180) (unit 1)
     (in_bom yes) (on_board yes) (fields_autoplaced)
@@
     (pin "1")
   )
+  (symbol (lib_id "power:GND") (at 124.46 152.4 0) (unit 1)
+    (in_bom yes) (on_board yes)
+    (property "Reference" "#PWR0105" (id 0) (at 124.46 158.75 0)
+      (effects (font (size 1.27 1.27)) hide)
+    )
+    (property "Value" "GND" (id 1) (at 124.46 157.48 0))
+    (property "Footprint" "" (id 2) (at 124.46 152.4 0)
+      (effects (font (size 1.27 1.27)) hide)
+    )
+    (property "Datasheet" "" (id 3) (at 124.46 152.4 0)
+      (effects (font (size 1.27 1.27)) hide)
+    )
+    (pin "1")
+  )
   (symbol (lib_id "Transistor_FET:IRLB8721PBF") (at 293.37 74.93 0) (unit 1)
     (in_bom yes) (on_board yes) (fields_autoplaced)
@@
       (reference "#PWR05") (unit 1) (value "+5V") (footprint "")
     )
-    (path "/01e4fccf-8023-47c5-8ebf-902e6ed6b0a3"
-      (reference "#PWR06") (unit 1) (value "GND") (footprint "")
-    )
     (path "/c8388099-9606-46b9-9f66-ad2ea4b72ec6/a8f4949d-a997-4597-bd13-164ec0d8afb8"
       (reference "#PWR07") (unit 1) (value "+12V") (footprint "")
@@
       (reference "#PWR0104") (unit 1) (value "+5V") (footprint "")
     )
-    (path "/c8388099-9606-46b9-9f66-ad2ea4b72ec6/3bedd05b-2dac-4928-b481-4e94d1fc07be"
+    (path "/febb5532-f50b-4206-9c76-51e32fa8cfdc"
       (reference "#PWR0105") (unit 1) (value "GND") (footprint "")
     )
@@
       (reference "C2") (unit 1) (value "0.01 μf") (footprint "Capacitor_THT:C_Disc_D3.0mm_W1.6mm_P2.50mm")
     )
-    (path "/c8388099-9606-46b9-9f66-ad2ea4b72ec6/04ce182a-7abb-4f82-b92f-59beb92690a5"
-      (reference "C3") (unit 1) (value "220uF") (footprint "Capacitor_THT:CP_Radial_D6.3mm_P2.50mm")
+    (path "/c8388099-9606-46b9-9f66-ad2ea4b72ec6/0567ebc0-6b29-4900-b5b8-9c8a8ac19768"
+      (reference "C3") (unit 1) (value "100nF") (footprint "Capacitor_THT:C_Disc_D4.7mm_W2.5mm_P5.00mm")
     )
     (path "/c8388099-9606-46b9-9f66-ad2ea4b72ec6/09c80e56-2dd2-46de-971b-4f170f74a8c6"
@@
       (reference "U3") (unit 1) (value "L298HN") (footprint "Package_TO_SOT_THT:TO-220-15_P2.54x2.54mm_StaggerOdd_Lead4.58mm_Vertical")
     )
-    (path "/c8388099-9606-46b9-9f66-ad2ea4b72ec6/6903a76f-65b1-46d9-9725-712dbf64ad32"
-      (reference "U4") (unit 1) (value "WS78L10") (footprint "Nick:TO-92L_Inline_China")
+    (path "/c8388099-9606-46b9-9f66-ad2ea4b72ec6/2bb05439-fb20-45a4-b0f5-c7ae48a3d511"
+      (reference "U4") (unit 1) (value "L7810") (footprint "")
     )
   )

Commit message: Add reverse voltage diode and re-draw ground plane
Parts:
- added D2: 1N4001, Diode_THT:D_DO-41_SOD81_P10.16mm_Horizontal, symbol Device:D_Schottky
- added J4: Pluggable_Terminal_01x02, TerminalBlock_Phoenix:TerminalBlock_Phoenix_MKDS-1,5-2-5.08_1x02_P5.08mm_Horizontal, symbol Connector:Screw_Terminal_01x02
- renumbered D2 to D3, D3 to D4, D4 to D5, D5 to D6, D6 to D7, D7 to D8, D8 to D9, J9 to J10, J10 to J11, J4 to J5, J5 to J6, J6 to J7, J7 to J8, J8 to J9, R11 to R10, R12 to R11, R13 to R12, R14 to R13, R15 to R14, R16 to R15, R17 to R16, R18 to R17, R19 to R18, R20 to R19, R21 to R20, R22 to R21, R9 to R8, R10 to R9
Connections:
- net BattRelayNC_Coil renamed BattRelayNC_Coil_A
- net BattRelayNC_Coil_A: now also D2.1 (K), J4.1 (Pin_1); no longer D4.1 (K), J5.4 (Pin_4), Q1.3 (D)
- new net BattRelayNC_Coil_B: D2.2 (A), D4.1 (K), J4.2 (Pin_2), Q1.3 (D)
Other:
- note added: "Prototype TODO: - Add reverse voltage protection diode to battery relay - Check all R values - Test current on each SR out (max 20mA, limit 35mA) - Test current on SR VCC (max 70mA)"
- note added: "Schematic TODO: - Disable SR when no input voltage (SR can draw power from inputs; i.e. MC) - Consider adding reverse voltage protection to power outputs - Check if PSU relay module has reverse voltage diode"
- note removed: "Prototype TODO: - Swithc out L7805 for L7810 (motor driver supply FET driver) - Check all R values - Test current on each SR out (max 20mA, limit 35mA) - Test current on SR VCC (max 70mA)"
- note removed: "Schematic TODO: - Disable SR when no input voltage (SR can draw power from inputs; i.e. MC)"
