File: hardware/greenhouse-node/_autosave-greenhouse-node-motor.kicad_sch (KiCad schematic)
At the start: 20 parts, among them J7 Conn_01x02_Male, Q2 2N2222A, Q4 IRF9530N, Q5 IRF530N, Q6 FDP7030DL, Q7 IRF9530N, Q8 IRF530N, U4 L7810

Commit message: Reduced NPN count
Parts:
- gave numbers to parts that had none: 4
- renumbered Q4 to Q3, Q5 to Q4, Q6 to Q5, Q7 to Q6, Q8 to Q7, R14 to R12, R15 to R13, R10 to R9
Changed lines of the file:
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@@
   (symbol (lib_id "power:+12V") (at 127 53.34 0) (unit 1)
     (in_bom yes) (on_board yes) (fields_autoplaced)
-    (property "Reference" "#PWR027" (id 0) (at 127 57.15 0)
+    (property "Reference" "#PWR026" (id 0) (at 127 57.15 0)
       (effects (font (size 1.27 1.27)) hide)
     )
@@
   (symbol (lib_id "Nick:2N2222A") (at 137.16 130.81 0) (mirror y) (unit 1)
     (in_bom yes) (on_board yes) (fields_autoplaced)
-    (property "Reference" "Q?" (id 0) (at 132.08 129.5399 0)
+    (property "Reference" "Q8" (id 0) (at 132.08 129.5399 0)
       (effects (font (size 1.27 1.27)) (justify left))
     )
@@
   (symbol (lib_id "power:GND") (at 228.6 120.65 0) (unit 1)
     (in_bom yes) (on_board yes) (fields_autoplaced)
-    (property "Reference" "#PWR031" (id 0) (at 228.6 127 0)
+    (property "Reference" "#PWR029" (id 0) (at 228.6 127 0)
       (effects (font (size 1.27 1.27)) hide)
     )
@@
   (symbol (lib_id "Transistor_FET:IRF9540N") (at 95.25 100.33 0) (mirror x) (unit 1)
     (in_bom yes) (on_board yes) (fields_autoplaced)
-    (property "Reference" "Q4" (id 0) (at 101.6 99.0599 0)
+    (property "Reference" "Q3" (id 0) (at 101.6 99.0599 0)
       (effects (font (size 1.27 1.27)) (justify left))
     )
@@
   (symbol (lib_id "power:GND") (at 90.17 72.39 0) (unit 1)
     (in_bom yes) (on_board yes) (fields_autoplaced)
-    (property "Reference" "#PWR023" (id 0) (at 90.17 78.74 0)
+    (property "Reference" "#PWR022" (id 0) (at 90.17 78.74 0)
       (effects (font (size 1.27 1.27)) hide)
     )
@@
   (symbol (lib_id "power:+12V") (at 74.93 53.34 0) (unit 1)
     (in_bom yes) (on_board yes) (fields_autoplaced)
-    (property "Reference" "#PWR021" (id 0) (at 74.93 57.15 0)
+    (property "Reference" "#PWR020" (id 0) (at 74.93 57.15 0)
       (effects (font (size 1.27 1.27)) hide)
     )
@@
   (symbol (lib_id "power:+10V") (at 111.76 90.17 0) (unit 1)
     (in_bom yes) (on_board yes) (fields_autoplaced)
-    (property "Reference" "#PWR024" (id 0) (at 111.76 93.98 0)
+    (property "Reference" "#PWR023" (id 0) (at 111.76 93.98 0)
       (effects (font (size 1.27 1.27)) hide)
     )
@@
   (symbol (lib_id "Transistor_FET:IRF540N") (at 124.46 58.42 0) (unit 1)
     (in_bom yes) (on_board yes) (fields_autoplaced)
-    (property "Reference" "Q6" (id 0) (at 130.81 57.1499 0)
+    (property "Reference" "Q5" (id 0) (at 130.81 57.1499 0)
       (effects (font (size 1.27 1.27)) (justify left))
     )
@@
   (symbol (lib_id "Transistor_FET:IRF9540N") (at 128.27 100.33 180) (unit 1)
     (in_bom yes) (on_board yes) (fields_autoplaced)
-    (property "Reference" "Q7" (id 0) (at 121.92 99.0599 0)
+    (property "Reference" "Q6" (id 0) (at 121.92 99.0599 0)
       (effects (font (size 1.27 1.27)) (justify left))
     )
@@
   (symbol (lib_id "Transistor_FET:IRF540N") (at 95.25 119.38 0) (unit 1)
     (in_bom yes) (on_board yes) (fields_autoplaced)
-    (property "Reference" "Q5" (id 0) (at 101.6 118.1099 0)
+    (property "Reference" "Q4" (id 0) (at 101.6 118.1099 0)
       (effects (font (size 1.27 1.27)) (justify left))
     )
@@
   (symbol (lib_id "power:+10V") (at 144.78 59.69 0) (unit 1)
     (in_bom yes) (on_board yes) (fields_autoplaced)
-    (property "Reference" "#PWR029" (id 0) (at 144.78 63.5 0)
+    (property "Reference" "#PWR028" (id 0) (at 144.78 63.5 0)
       (effects (font (size 1.27 1.27)) hide)
     )
@@
   (symbol (lib_id "Device:R_Small_US") (at 143.51 125.73 180) (unit 1)
     (in_bom yes) (on_board yes) (fields_autoplaced)
-    (property "Reference" "R?" (id 0) (at 146.05 124.4599 0)
+    (property "Reference" "R11" (id 0) (at 146.05 124.4599 0)
       (effects (font (size 1.27 1.27)) (justify right))
     )
@@
   (symbol (lib_id "Device:R_Small_US") (at 88.9 96.52 180) (unit 1)
     (in_bom yes) (on_board yes) (fields_autoplaced)
-    (property "Reference" "R?" (id 0) (at 86.36 95.2499 0)
+    (property "Reference" "R8" (id 0) (at 86.36 95.2499 0)
       (effects (font (size 1.27 1.27)) (justify left))
     )
@@
   (symbol (lib_id "Device:R_Small_US") (at 134.62 96.52 0) (mirror x) (unit 1)
     (in_bom yes) (on_board yes) (fields_autoplaced)
-    (property "Reference" "R?" (id 0) (at 137.16 95.2499 0)
+    (property "Reference" "R10" (id 0) (at 137.16 95.2499 0)
       (effects (font (size 1.27 1.27)) (justify left))
     )
@@
   (symbol (lib_id "Device:R_Small_US") (at 114.3 60.96 0) (mirror x) (unit 1)
     (in_bom yes) (on_board yes) (fields_autoplaced)
-    (property "Reference" "R10" (id 0) (at 111.76 59.6899 0)
+    (property "Reference" "R9" (id 0) (at 111.76 59.6899 0)
       (effects (font (size 1.27 1.27)) (justify right))
     )
@@
   (symbol (lib_id "Device:R_Small_US") (at 220.98 116.84 270) (mirror x) (unit 1)
     (in_bom yes) (on_board yes) (fields_autoplaced)
-    (property "Reference" "R15" (id 0) (at 220.98 110.49 90))
+    (property "Reference" "R13" (id 0) (at 220.98 110.49 90))
     (property "Value" "5k" (id 1) (at 220.98 113.03 90))
     (property "Footprint" "Resistor_THT:R_Axial_DIN0204_L3.6mm_D1.6mm_P7.62mm_Horizontal" (id 2) (at 220.98 116.84 0)
@@
   (symbol (lib_id "Device:R_Small_US") (at 220.98 106.68 270) (mirror x) (unit 1)
     (in_bom yes) (on_board yes) (fields_autoplaced)
-    (property "Reference" "R14" (id 0) (at 220.98 100.33 90))
+    (property "Reference" "R12" (id 0) (at 220.98 100.33 90))
     (property "Value" "5k" (id 1) (at 220.98 102.87 90))
     (property "Footprint" "Resistor_THT:R_Axial_DIN0204_L3.6mm_D1.6mm_P7.62mm_Horizontal" (id 2) (at 220.98 106.68 0)
@@
   (symbol (lib_id "Transistor_FET:IRF540N") (at 128.27 119.38 0) (mirror y) (unit 1)
     (in_bom yes) (on_board yes) (fields_autoplaced)
-    (property "Reference" "Q8" (id 0) (at 121.92 118.1099 0)
+    (property "Reference" "Q7" (id 0) (at 121.92 118.1099 0)
       (effects (font (size 1.27 1.27)) (justify left))
     )
@@
   (symbol (lib_id "power:GND") (at 114.3 63.5 0) (mirror y) (unit 1)
     (in_bom yes) (on_board yes)
-    (property "Reference" "#PWR026" (id 0) (at 114.3 69.85 0)
+    (property "Reference" "#PWR025" (id 0) (at 114.3 69.85 0)
       (effects (font (size 1.27 1.27)) hide)
     )
@@
   (symbol (lib_id "power:GND") (at 111.76 135.89 0) (unit 1)
     (in_bom yes) (on_board yes)
-    (property "Reference" "#PWR025" (id 0) (at 111.76 142.24 0)
+    (property "Reference" "#PWR024" (id 0) (at 111.76 142.24 0)
       (effects (font (size 1.27 1.27)) hide)
     )
@@
   (symbol (lib_id "power:GND") (at 88.9 135.89 0) (unit 1)
     (in_bom yes) (on_board yes) (fields_autoplaced)
-    (property "Reference" "#PWR020" (id 0) (at 88.9 142.24 0)
+    (property "Reference" "#PWR021" (id 0) (at 88.9 142.24 0)
       (effects (font (size 1.27 1.27)) hide)
     )
@@
   (symbol (lib_id "power:GND") (at 134.62 135.89 0) (mirror y) (unit 1)
     (in_bom yes) (on_board yes) (fields_autoplaced)
-    (property "Reference" "#PWR?" (id 0) (at 134.62 142.24 0)
-      (effects (font (size 1.27 1.27)) hide)
-    )
+    (property "Reference" "#PWR027" (id 0) (at 134.62 142.24 0)
+      (effects (font (size 1.27 1.27)) hide)
+    )
