File: hardware/greenhouse-node/greenhouse-node.kicad_sch (KiCad schematic)
At the start: 28 parts, among them J1 Conn_01x04_Male, J2 Conn_01x12_Male, J3 Conn_01x02_Male, J4 Conn_01x02_Male, J5 RX_PinHeader_1x04_P2.54mm, J6 TX_PinHeader_1x04_P2.54mm, Q1 BC549C, U1 ATtiny84A-P, U2 L7805, U3 74HC595

Commit message: Remove voltage regulator
Provide +10V with buck converter instead; perhaps regulate actuator with PWM to control speed
Connections:
- net +12V renamed +10V
Changed lines of the file:
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@@
     (pin "2")
-  )
-  (symbol (lib_id "power:+12V") (at 60.96 30.48 0) (unit 1)
-    (in_bom yes) (on_board yes) (fields_autoplaced)
-    (property "Reference" "#PWR04" (id 0) (at 60.96 34.29 0)
-      (effects (font (size 1.27 1.27)) hide)
-    )
-    (property "Value" "+12V" (id 1) (at 60.96 25.4 0))
-    (property "Footprint" "" (id 2) (at 60.96 30.48 0)
-      (effects (font (size 1.27 1.27)) hide)
-    )
-    (property "Datasheet" "" (id 3) (at 60.96 30.48 0)
-      (effects (font (size 1.27 1.27)) hide)
-    )
-    (pin "1")
   )
   (symbol (lib_id "power:GND") (at 179.07 67.31 0) (unit 1)
@@
     (pin "2")
   )
+  (symbol (lib_id "power:+10V") (at 92.71 39.37 0) (unit 1)
+    (in_bom yes) (on_board yes) (fields_autoplaced)
+    (property "Reference" "#PWR0102" (id 0) (at 92.71 43.18 0)
+      (effects (font (size 1.27 1.27)) hide)
+    )
+    (property "Value" "+10V" (id 1) (at 92.71 34.29 0))
+    (property "Footprint" "" (id 2) (at 92.71 39.37 0)
+      (effects (font (size 1.27 1.27)) hide)
+    )
+    (property "Datasheet" "" (id 3) (at 92.71 39.37 0)
+      (effects (font (size 1.27 1.27)) hide)
+    )
+    (pin "1")
+  )
   (symbol (lib_id "Device:R_Small_US") (at 172.72 53.34 270) (mirror x) (unit 1)
     (in_bom yes) (on_board yes) (fields_autoplaced)
@@
     )
     (property "Datasheet" "" (id 3) (at 134.62 90.17 0)
+      (effects (font (size 1.27 1.27)) hide)
+    )
+    (pin "1")
+  )
+  (symbol (lib_id "power:+10V") (at 60.96 30.48 0) (unit 1)
+    (in_bom yes) (on_board yes) (fields_autoplaced)
+    (property "Reference" "#PWR0101" (id 0) (at 60.96 34.29 0)
+      (effects (font (size 1.27 1.27)) hide)
+    )
+    (property "Value" "+10V" (id 1) (at 60.96 25.4 0))
+    (property "Footprint" "" (id 2) (at 60.96 30.48 0)
+      (effects (font (size 1.27 1.27)) hide)
+    )
+    (property "Datasheet" "" (id 3) (at 60.96 30.48 0)
       (effects (font (size 1.27 1.27)) hide)
     )
@@
     (pin "2")
   )
-  (symbol (lib_id "power:+12V") (at 92.71 39.37 0) (unit 1)
-    (in_bom yes) (on_board yes) (fields_autoplaced)
-    (property "Reference" "#PWR07" (id 0) (at 92.71 43.18 0)
-      (effects (font (size 1.27 1.27)) hide)
-    )
-    (property "Value" "+12V" (id 1) (at 92.71 34.29 0))
-    (property "Footprint" "" (id 2) (at 92.71 39.37 0)
-      (effects (font (size 1.27 1.27)) hide)
-    )
-    (property "Datasheet" "" (id 3) (at 92.71 39.37 0)
-      (effects (font (size 1.27 1.27)) hide)
-    )
-    (pin "1")
-  )
   (sheet (at 34.29 153.67) (size 36.83 30.48) (fields_autoplaced)
     (stroke (width 0.1524) (type solid) (color 0 0 0 0))
@@
       (reference "#PWR03") (unit 1) (value "GND") (footprint "")
     )
-    (path "/1e48e0ab-1b14-4d0d-bb77-ec49319e2d5a"
-      (reference "#PWR04") (unit 1) (value "+12V") (footprint "")
-    )
     (path "/d53640f8-290d-4818-9efa-fa16f9f28a47"
       (reference "#PWR05") (unit 1) (value "GND") (footprint "")
@@
       (reference "#PWR06") (unit 1) (value "GND") (footprint "")
     )
-    (path "/fe477825-6d62-48dc-bb28-b91964e89730"
-      (reference "#PWR07") (unit 1) (value "+12V") (footprint "")
-    )
     (path "/cbcb4db5-db5f-4238-b5e9-7c269f0aa1c5"
       (reference "#PWR08") (unit 1) (value "+5V") (footprint "")
@@
       (reference "#PWR019") (unit 1) (value "GND") (footprint "")
     )
-    (path "/f125db1d-864d-4c2f-aa44-ac14276ec569/42979d9c-45c7-44ea-b09e-664b9987e3cb"
-      (reference "#PWR020") (unit 1) (value "+12V") (footprint "")
-    )
     (path "/f125db1d-864d-4c2f-aa44-ac14276ec569/eb83045a-3265-4cb3-a640-fc71123b572b"
       (reference "#PWR021") (unit 1) (value "GND") (footprint "")
     )
-    (path "/f125db1d-864d-4c2f-aa44-ac14276ec569/4094f064-5398-4528-94a6-9af7303eefd2"
-      (reference "#PWR022") (unit 1) (value "GND") (footprint "")
-    )
     (path "/f125db1d-864d-4c2f-aa44-ac14276ec569/4555a28c-f6f1-4471-86dd-c79e1eb5f92d"
       (reference "#PWR023") (unit 1) (value "+10V") (footprint "")
@@
       (reference "#PWR024") (unit 1) (value "GND") (footprint "")
     )
-    (path "/f125db1d-864d-4c2f-aa44-ac14276ec569/e3c32dad-56ae-40c1-b262-607020b74545"
-      (reference "#PWR025") (unit 1) (value "GND") (footprint "")
-    )
-    (path "/f125db1d-864d-4c2f-aa44-ac14276ec569/0b9c82ff-229c-4ba3-86ae-ce5fc883bef6"
-      (reference "#PWR026") (unit 1) (value "+12V") (footprint "")
-    )
     (path "/f125db1d-864d-4c2f-aa44-ac14276ec569/faa75408-7bc9-47b9-8a84-b71947d6e554"
       (reference "#PWR027") (unit 1) (value "GND") (footprint "")
     )
-    (path "/f125db1d-864d-4c2f-aa44-ac14276ec569/7edb6214-ff1b-45cd-bece-105eb508f1e9"
-      (reference "#PWR028") (unit 1) (value "+10V") (footprint "")
+    (path "/8d1f2d93-6b8f-4b97-be35-6dc31d235797"
+      (reference "#PWR0101") (unit 1) (value "+10V") (footprint "")
+    )
+    (path "/4084c646-f815-4943-8f01-85c8a25567cf"
+      (reference "#PWR0102") (unit 1) (value "+10V") (footprint "")
     )
     (path "/1bbe0bee-1018-4ce9-bd17-02581403417d"
@@
       (reference "C4") (unit 1) (value "10nF") (footprint "Capacitor_THT:C_Disc_D4.7mm_W2.5mm_P5.00mm")
     )
-    (path "/f125db1d-864d-4c2f-aa44-ac14276ec569/f62ed550-59dc-4b33-bb48-0dfd67d12b7c"
-      (reference "C5") (unit 1) (value "330nF") (footprint "Capacitor_THT:C_Disc_D4.7mm_W2.5mm_P5.00mm")
-    )
-    (path "/f125db1d-864d-4c2f-aa44-ac14276ec569/37ff04cd-08d4-4a19-a627-432ceb192578"
-      (reference "C6") (unit 1) (value "100nF") (footprint "Capacitor_THT:C_Disc_D4.7mm_W2.5mm_P5.00mm")
-    )
     (path "/51b7deb3-d546-4266-aa92-b89ded074dd4"
       (reference "D1") (unit 1) (value "LED_Small") (footprint "LED_THT:LED_D3.0mm")
@@
       (reference "Q4") (unit 1) (value "IRF530N") (footprint "Package_TO_SOT_THT:TO-220-3_Horizontal_TabDown")
     )
-    (path "/f125db1d-864d-4c2f-aa44-ac14276ec569/4776eb62-0319-43f7-a210-29442a9c84c1"
-      (reference "Q5") (unit 1) (value "FDP7030DL") (footprint "Package_TO_SOT_THT:TO-220-3_Horizontal_TabDown")
-    )
     (path "/f125db1d-864d-4c2f-aa44-ac14276ec569/6ea00187-9c84-4f7e-91e0-78d37efe1b8e"
       (reference "Q6") (unit 1) (value "IRF9530N") (footprint "Package_TO_SOT_THT:TO-220-3_Horizontal_TabDown")
@@
       (reference "R8") (unit 1) (value "10k") (footprint "Resistor_THT:R_Axial_DIN0204_L3.6mm_D1.6mm_P7.62mm_Horizontal")
     )
-    (path "/f125db1d-864d-4c2f-aa44-ac14276ec569/d33d0fb3-6d1f-4cc7-b00d-5d21fba58dee"
-      (reference "R9") (unit 1) (value "10k") (footprint "Resistor_THT:R_Axial_DIN0204_L3.6mm_D1.6mm_P7.62mm_Horizontal")
-    )
     (path "/f125db1d-864d-4c2f-aa44-ac14276ec569/bf817e6d-58a1-41ad-a248-45e7818135e2"
       (reference "R10") (unit 1) (value "10k") (footprint "Resistor_THT:R_Axial_DIN0204_L3.6mm_D1.6mm_P7.62mm_Horizontal")
@@
       (reference "U3") (unit 1) (value "74HC595") (footprint "Package_DIP:DIP-16_W7.62mm_Socket")
     )
-    (path "/f125db1d-864d-4c2f-aa44-ac14276ec569/47180113-64b9-40b2-a38e-b438f63a3376"
-      (reference "U4") (unit 1) (value "L7810") (footprint "Nick:TO-92L_Inline_Regulator")
-    )
-  )
+  )
