File: hardware/greenhouse-node/greenhouse-node-motor.kicad_sch (KiCad schematic)
At the start: 19 parts, among them J8 Conn_01x02_Male, Q2 BC549C, Q3 BC549C, Q4 IRF9530N, Q5 IRF530N, Q6 IRF9530N, Q7 IRF530N, Q8 BC549C, Q9 BC549C

Commit message: Add cap and diode
Parts:
- renumbered D5 to D6, D6 to D7
Changed lines of the file:
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@@
   (symbol (lib_name "LED_Small_1") (lib_id "Device:LED_Small") (at 196.85 120.65 180) (unit 1)
     (in_bom yes) (on_board yes) (fields_autoplaced)
-    (property "Reference" "D5" (id 0) (at 196.7865 114.3 0))
+    (property "Reference" "D6" (id 0) (at 196.7865 114.3 0))
     (property "Value" "LED_Sm_B" (id 1) (at 196.7865 116.84 0))
     (property "Footprint" "LED_THT:LED_D3.0mm" (id 2) (at 196.85 120.65 90)
@@
   (symbol (lib_id "Device:LED_Small") (at 196.85 130.81 180) (unit 1)
     (in_bom yes) (on_board yes) (fields_autoplaced)
-    (property "Reference" "D6" (id 0) (at 196.7865 124.46 0))
+    (property "Reference" "D7" (id 0) (at 196.7865 124.46 0))
     (property "Value" "LED_Sm_Y" (id 1) (at 196.7865 127 0))
     (property "Footprint" "LED_THT:LED_D3.0mm" (id 2) (at 196.85 130.81 90)
